File: design/D8-2L-FASTON/MAIN_POWER/MAIN_POWER.kicad_pcb (KiCad board)
At the start: 2 copper layers, 121.8 x 60.5 mm, 17 parts, among them J1 12V INPUT - FASTON 250, J2 JETSON 12V 5A, J3 GMSL 12V / EXCLUSIVE WITH POE, J4 FAN 12V 0.14A, J5 USB BOARD 12V, J6 POE BOARD 12V INPUT

Commit message: Apply MAIN V3 outline and export FASTON STEP
Parts:
- moved J1 3.43 mm to (139.6, 108.8)
- moved H2 3.00 mm to (123.6, 59.1)
- moved H5 3.00 mm to (155.6, 59.1)
Other:
- outline, holes or cut-outs redrawn
- board text removed: "J1: +12V / GND SOLDER PADS"
Changed lines of the file:
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@@
 	(footprint "UMI_D2:MountingHole_3.5mm"
 		(layer "F.Cu")
-		(at 120.6 59.131981)
+		(at 123.6 59.131981)
 		(property "Reference" "H2"
 			(at 0 -3 0)
@@
 			)
 		)
+		(property "MPN" "MECHANICAL - NO PURCHASE"
+			(at 0 0 0)
+			(layer "F.Fab")
+			(hide yes)
+			(effects
+				(font
+					(size 1 1)
+					(thickness 0.15)
+				)
+			)
+		)
 		(attr exclude_from_pos_files exclude_from_bom)
 		(duplicate_pad_numbers_are_jumpers no)
@@
 	(footprint "UMI_D2:MountingHole_3.5mm"
 		(layer "F.Cu")
-		(at 158.6 59.131981)
+		(at 155.6 59.131981)
 		(property "Reference" "H5"
 			(at 0 -3 0)
@@
 			)
 		)
+		(property "MPN" "MECHANICAL - NO PURCHASE"
+			(at 0 0 0)
+			(layer "F.Fab")
+			(hide yes)
+			(effects
+				(font
+					(size 1 1)
+					(thickness 0.15)
+				)
+			)
+		)
 		(attr exclude_from_pos_files exclude_from_bom)
 		(duplicate_pad_numbers_are_jumpers no)
@@
 			)
 		)
+		(property "MPN" "MECHANICAL - NO PURCHASE"
+			(at 0 0 0)
+			(layer "F.Fab")
+			(hide yes)
+			(effects
+				(font
+					(size 1 1)
+					(thickness 0.15)
+				)
+			)
+		)
 		(attr exclude_from_pos_files exclude_from_bom)
 		(duplicate_pad_numbers_are_jumpers no)
@@
 			)
 		)
+		(property "MPN" "MECHANICAL - NO PURCHASE"
+			(at 0 0 0)
+			(layer "F.Fab")
+			(hide yes)
+			(effects
+				(font
+					(size 1 1)
+					(thickness 0.15)
+				)
+			)
+		)
 		(attr exclude_from_pos_files exclude_from_bom)
 		(duplicate_pad_numbers_are_jumpers no)
@@
 		)
 		(embedded_fonts no)
-		(model "${KICAD6_3DMODEL_DIR}/Connector_JST.3dshapes/JST_VH_B2P-VH_1x02_P3.96mm_Vertical.wrl"
+		(model "${KICAD6_3DMODEL_DIR}/Connector_JST.3dshapes/JST_EH_B2B-EH-A_1x02_P2.50mm_Vertical.step"
 			(offset
 				(xyz 0 0 0)
@@
 		)
 		(embedded_fonts no)
-		(model "${KICAD6_3DMODEL_DIR}/Connector_JST.3dshapes/JST_VH_B2P-VH_1x02_P3.96mm_Vertical.wrl"
+		(model "${KICAD6_3DMODEL_DIR}/Connector_JST.3dshapes/JST_EH_B2B-EH-A_1x02_P2.50mm_Vertical.step"
 			(offset
 				(xyz 0 0 0)
@@
 		)
 		(embedded_fonts no)
-		(model "${KICAD6_3DMODEL_DIR}/Connector_JST.3dshapes/JST_VH_B2P-VH_1x02_P3.96mm_Vertical.wrl"
+		(model "${KICAD6_3DMODEL_DIR}/Connector_JST.3dshapes/JST_EH_B2B-EH-A_1x02_P2.50mm_Vertical.step"
 			(offset
 				(xyz 0 0 0)
@@
 		)
 		(embedded_fonts no)
-		(model "${KICAD6_3DMODEL_DIR}/Connector_JST.3dshapes/JST_VH_B2P-VH_1x02_P3.96mm_Vertical.wrl"
+		(model "${KICAD6_3DMODEL_DIR}/Connector_JST.3dshapes/JST_EH_B2B-EH-A_1x02_P2.50mm_Vertical.step"
 			(offset
 				(xyz 0 0 0)
@@
 			)
 		)
+		(property "MPN" "MECHANICAL - NO PURCHASE"
+			(at 0 0 0)
+			(layer "F.Fab")
+			(hide yes)
+			(effects
+				(font
+					(size 1 1)
+					(thickness 0.15)
+				)
+			)
+		)
 		(attr exclude_from_pos_files exclude_from_bom)
 		(duplicate_pad_numbers_are_jumpers no)
@@
 		)
 		(embedded_fonts no)
-		(model "${KICAD6_3DMODEL_DIR}/Connector_JST.3dshapes/JST_VH_B2P-VH_1x02_P3.96mm_Vertical.wrl"
+		(model "${KICAD6_3DMODEL_DIR}/Connector_JST.3dshapes/JST_EH_B2B-EH-A_1x02_P2.50mm_Vertical.step"
 			(offset
 				(xyz 0 0 0)
@@
 		)
 	)
-	(footprint "UMI_D2:MountingHole_3.5mm"
-		(layer "F.Cu")
-		(at 82.7 76.610156)
-		(property "Reference" "H1"
-			(at 0 -3 0)
-			(layer "F.Fab")
-			(hide yes)
-			(effects
-				(font
-					(size 1 1)
-					(thickness 0.15)
-				)
-			)
-		)
-		(property "Value" "DXF 3.5mm NPTH"
-			(at 0 3 0)
-			(layer "F.Fab")
-			(hide yes)
-			(effects
-				(font
-					(size 1 1)
-					(thickness 0.15)
-				)
-			)
-		)
-		(property "Datasheet" ""
-			(at 0 0 0)
-			(layer "F.Fab")
-			(hide yes)
-			(effects
-				(font
-					(size 1.27 1.27)
-				)
-			)
-		)
-		(property "Description" ""
-			(at 0 0 0)
-			(layer "F.Fab")
-			(hide yes)
-			(effects
-				(font
-					(size 1.27 1.27)
-				)
-			)
-		)
-		(attr exclude_from_pos_files exclude_from_bom)
-		(duplicate_pad_numbers_are_jumpers no)
-		(pad "" np_thru_hole circle
-			(at 0 0)
-			(size 3.5 3.5)
-			(drill 3.5)
-			(layers "*.Cu" "*.Mask")
-		)
-		(embedded_fonts no)
-	)
 	(footprint "UMI_D2:Input_FASTON_250_PAIR"
 		(layer "F.Cu")
-		(at 137.9 105.85)
+		(at 139.6 108.832)
 		(descr "Two TE Connectivity FASTON 250 PCB tabs, 63951-4; two 1.4 mm plated holes per tab at 5.08 mm pitch; blades toward top")
 		(tags "FASTON 250 63951-4 input 12V")
@@
 		)
 		(embedded_fonts no)
+		(model "${KIPRJMOD}/3d/FASTON_63951-4_PAIR_PROXY.step"
+			(offset
+				(xyz 0 0 0)
+			)
+			(scale
+				(xyz 1 1 1)
+			)
+			(rotate
+				(xyz 0 0 0)
+			)
+		)
+	)
+	(footprint "UMI_D2:MountingHole_3.5mm"
+		(layer "F.Cu")
+		(at 82.7 76.610156)
+		(property "Reference" "H1"
+			(at 0 -3 0)
+			(layer "F.Fab")
+			(hide yes)
+			(effects
+				(font
+					(size 1 1)
+					(thickness 0.15)
+				)
+			)
+		)
+		(property "Value" "DXF 3.5mm NPTH"
+			(at 0 3 0)
+			(layer "F.Fab")
+			(hide yes)
+			(effects
+				(font
+					(size 1 1)
+					(thickness 0.15)
+				)
+			)
+		)
+		(property "Datasheet" ""
+			(at 0 0 0)
+			(layer "F.Fab")
+			(hide yes)
+			(effects
+				(font
+					(size 1.27 1.27)
+				)
+			)
+		)
+		(property "Description" ""
+			(at 0 0 0)
+			(layer "F.Fab")
+			(hide yes)
+			(effects
+				(font
+					(size 1.27 1.27)
+				)
+			)
+		)
+		(property "MPN" "MECHANICAL - NO PURCHASE"
+			(at 0 0 0)
+			(layer "F.Fab")
+			(hide yes)
+			(effects
+				(font
+					(size 1 1)
+					(thickness 0.15)
+				)
+			)
+		)
+		(attr exclude_from_pos_files exclude_from_bom)
+		(duplicate_pad_numbers_are_jumpers no)
+		(pad "" np_thru_hole circle
+			(at 0 0)
+			(size 3.5 3.5)
+			(drill 3.5)
+			(layers "*.Cu" "*.Mask")
+		)
+		(embedded_fonts no)
 	)
 	(footprint "UMI_D2:FuseHolder_Blade_ATO_Littelfuse_FLR_178.6165"
@@
 		)
 		(embedded_fonts no)
-		(model "${KICAD7_3DMODEL_DIR}/Fuse.3dshapes/FuseHolder_Blade_ATO_Littelfuse_FLR_178.6165.wrl"
+		(model "${KICAD7_3DMODEL_DIR}/Fuse.3dshapes/Fuseholder_Blade_Mini_Keystone_3568.step"
 			(offset
 				(xyz 0 0 0)
@@
 		)
 		(embedded_fonts no)
-		(model "${KICAD7_3DMODEL_DIR}/Fuse.3dshapes/FuseHolder_Blade_ATO_Littelfuse_FLR_178.6165.wrl"
+		(model "${KICAD7_3DMODEL_DIR}/Fuse.3dshapes/Fuseholder_Blade_Mini_Keystone_3568.step"
 			(offset
 				(xyz 0 0 0)
@@
 		)
 		(embedded_fonts no)
-		(model "${KICAD7_3DMODEL_DIR}/Fuse.3dshapes/FuseHolder_Blade_ATO_Littelfuse_FLR_178.6165.wrl"
+		(model "${KICAD7_3DMODEL_DIR}/Fuse.3dshapes/Fuseholder_Blade_Mini_Keystone_3568.step"
 			(offset
 				(xyz 0 0 0)
@@
 		)
 		(embedded_fonts no)
-		(model "${KICAD7_3DMODEL_DIR}/Fuse.3dshapes/FuseHolder_Blade_ATO_Littelfuse_FLR_178.6165.wrl"
+		(model "${KICAD7_3DMODEL_DIR}/Fuse.3dshapes/Fuseholder_Blade_Mini_Keystone_3568.step"
 			(offset
 				(xyz 0 0 0)
@@
 		)
 		(embedded_fonts no)
-		(model "${KICAD7_3DMODEL_DIR}/Fuse.3dshapes/FuseHolder_Blade_ATO_Littelfuse_FLR_178.6165.wrl"
+		(model "${KICAD7_3DMODEL_DIR}/Fuse.3dshapes/Fuseholder_Blade_Mini_Keystone_3568.step"
 			(offset
 				(xyz 0 0 0)
@@
 		(layer "Edge.Cuts")
 	)
+	(gr_arc
+		(start 122.6 115.631981)
+		(mid 120.478686 114.7533)
+		(end 119.6 112.631981)
+		(stroke
+			(width 0.05)
+			(type solid)
+		)
+		(layer "Edge.Cuts")
+	)
 	(gr_line
-		(start 121.6 55.131981)
-		(end 89.156349 55.131981)
+		(start 122.6 115.631981)
+		(end 156.6 115.631981)
 		(stroke
 			(width 0.05)
@@
 		(layer "Edge.Cuts")
 	)
-	(gr_arc
-		(start 121.6 55.131981)
-		(mid 123.721327 56.01066)
-		(end 124.6 58.131981)
+	(gr_line
+		(start 123.6 55.131981)
+		(end 89.156349 55.131981)
 		(stroke
 			(width 0.05)
@@
 	)
 	(gr_arc
-		(start 122.6 115.631981)
-		(mid 120.478686 114.7533)
-		(end 119.6 112.631981)
+		(start 123.6 55.131981)
+		(mid 127.416439 57.934155)
+		(end 125.885714 62.414588)
 		(stroke
 			(width 0.05)
@@
 		(layer "Edge.Cuts")
 	)
-	(gr_line
-		(start 122.6 115.631981)
-		(end 156.6 115.631981)
+	(gr_arc
+		(start 124.6 64.876544)
+		(mid 124.940768 63.487801)
+		(end 125.885714 62.414589)
 		(stroke
 			(width 0.05)
@@
 	(gr_line
 		(start 124.6 69.131981)
-		(end 124.6 58.131981)
+		(end 124.6 64.876544)
 		(stroke
 			(width 0.05)
@@
 		(layer "Edge.Cuts")
 	)
-	(gr_line
-		(start 154.6 58.131981)
-		(end 154.6 69.131981)
+	(gr_arc
+		(start 153.314286 62.414589)
+		(mid 154.2592 63.487818)
+		(end 154.6 64.876544)
 		(stroke
 			(width 0.05)
@@
 	)
 	(gr_arc
-		(start 154.6 58.131981)
-		(mid 155.478686 56.010673)
-		(end 157.6 55.131981)
+		(start 153.314286 62.414588)
+		(mid 151.783577 57.934174)
+		(end 155.6 55.131981)
+		(stroke
+			(width 0.05)
+			(type solid)
+		)
+		(layer "Edge.Cuts")
+	)
+	(gr_line
+		(start 154.6 64.876544)
+		(end 154.6 69.131981)
 		(stroke
 			(width 0.05)
@@
 	)
 	(gr_line
-		(start 168.72132 91.510661)
-		(end 160.47868 99.753301)
+		(start 160.47868 99.753301)
+		(end 168.72132 91.510661)
 		(stroke
 			(width 0.05)
@@
 	(gr_line
 		(start 190.043651 55.131981)
-		(end 157.6 55.131981)
+		(end 155.6 55.131981)
 		(stroke
 			(width 0.05)
@@
 		)
 	)
-	(gr_text "J1: +12V / GND SOLDER PADS"
-		(at 140 108.65 0)
-		(layer "F.SilkS")
-		(effects
-			(font
-				(size 1.1 1.1)
-				(thickness 0.15)
-			)
-		)
-	)
 	(gr_text "UMI 12V DISTRIBUTION"
 		(at 47 84 90)
@@
 	)
 	(group ""
-		(members "086dc82d-2124-5af7-8177-e6cf1e0a1d92" "5fb821b0-0cc2-5f1d-a01a-ba347644ca2b"
-			"7915ba4f-4c40-56c9-a00a-825aadb85623"
-		)
+		(members "086dc82d-2124-5af7-8177-e6cf1e0a1d92" "7915ba4f-4c40-56c9-a00a-825aadb85623")
 	)
 	(embedded_fonts no)
