File: design/D8-2L-FASTON/MAIN_POWER/MAIN_POWER.kicad_sch (KiCad schematic)
At the start: 15 parts, among them J1 12V INPUT - FASTON 250, J2 JETSON 12V 5A, J3 GMSL 12V / EXCLUSIVE WITH POE, J4 FAN 12V 0.14A, J5 USB BOARD 12V, J6 POE BOARD 12V INPUT

Commit message: Apply MAIN V3 outline and export FASTON STEP
Parts:
- added H5, H6: DXF 3.5mm NPTH, UMI_D2:MountingHole_3.5mm, symbol UMI:P_H4
- H1, H2, H3, H4: value M3 MOUNT -> DXF 3.5mm NPTH; footprint UMI_D2:MountingHole_4.5mm -> UMI_D2:MountingHole_3.5mm
Changed lines of the file:
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@@
     (property
       "Value"
-      "M3 MOUNT"
+      "DXF 3.5mm NPTH"
       (at 30.48 177.99 0)
       (effects
@@
     (property
       "Footprint"
-      "UMI_D2:MountingHole_4.5mm"
+      "UMI_D2:MountingHole_3.5mm"
       (at 30.48 173.99 0)
       (effects
@@
     (property
       "Value"
-      "M3 MOUNT"
+      "DXF 3.5mm NPTH"
       (at 50.8 177.99 0)
       (effects
@@
     (property
       "Footprint"
-      "UMI_D2:MountingHole_4.5mm"
+      "UMI_D2:MountingHole_3.5mm"
       (at 50.8 173.99 0)
       (effects
@@
     (property
       "Value"
-      "M3 MOUNT"
+      "DXF 3.5mm NPTH"
       (at 71.12 177.99 0)
       (effects
@@
     (property
       "Footprint"
-      "UMI_D2:MountingHole_4.5mm"
+      "UMI_D2:MountingHole_3.5mm"
       (at 71.12 173.99 0)
       (effects
@@
     (property
       "Value"
-      "M3 MOUNT"
+      "DXF 3.5mm NPTH"
       (at 91.44 177.99 0)
       (effects
@@
     (property
       "Footprint"
-      "UMI_D2:MountingHole_4.5mm"
+      "UMI_D2:MountingHole_3.5mm"
       (at 91.44 173.99 0)
       (effects
@@
           (unit 1)
         )
+      )
+    )
+  )
+  (symbol
+    (lib_id "UMI:P_H4")
+    (at 111.76 173.99 0)
+    (unit 1)
+    (in_bom no)
+    (on_board yes)
+    (dnp no)
+    (property
+      "Reference"
+      "H5"
+      (at 91.44 167.64 0)
+      (effects
+        (font
+          (size 1 1)
+        )
+      )
+    )
+    (property
+      "Value"
+      "DXF 3.5mm NPTH"
+      (at 91.44 177.99 0)
+      (effects
+        (font
+          (size 1 1)
+        )
+      )
+    )
+    (property
+      "Footprint"
+      "UMI_D2:MountingHole_3.5mm"
+      (at 111.76 173.99 0)
+      (effects
+        (font
+          (size 1 1)
+        )
+        hide
+      )
+    )
+    (property
+      "MPN"
+      "MECHANICAL - NO PURCHASE"
+      (at 111.76 173.99 0)
+      (effects
+        (font
+          (size 1 1)
+        )
+        hide
+      )
+    )
+    (instances
+      (project
+        "MAIN_POWER"
+        (path
+          "/71ea73aa-ccde-58dc-85f1-fbe1a59edb87"
+          (reference "H5")
+          (unit 1)
+        )
+      )
+    )
+  )
+  (symbol
+    (lib_id "UMI:P_H4")
+    (at 132.08 173.99 0)
+    (unit 1)
+    (in_bom no)
+    (on_board yes)
+    (dnp no)
+    (property
+      "Reference"
+      "H6"
+      (at 91.44 167.64 0)
+      (effects
+        (font
+          (size 1 1)
+        )
+      )
+    )
+    (property
+      "Value"
+      "DXF 3.5mm NPTH"
+      (at 91.44 177.99 0)
+      (effects
+        (font
+          (size 1 1)
+        )
+      )
+    )
+    (property
+      "Footprint"
+      "UMI_D2:MountingHole_3.5mm"
+      (at 132.08 173.99 0)
+      (effects
+        (font
+          (size 1 1)
+        )
+        hide
+      )
+    )
+    (property
+      "MPN"
+      "MECHANICAL - NO PURCHASE"
+      (at 132.08 173.99 0)
+      (effects
+        (font
+          (size 1 1)
+        )
+        hide
+      )
+    )
+    (instances
+      (project
+        "MAIN_POWER"
+        (path
+          "/71ea73aa-ccde-58dc-85f1-fbe1a59edb87"
+          (reference "H6")
+          (unit 1)
+        )
